File: 74141_subst.kicad_sch (KiCad schematic)
At the start: 14 parts, among them Q1 NHUMD12, Q2 NHUMD12, Q3 NHUMD12, Q4 NHUMD12, Q5 NHUMD12, U1 CD4028BPWR, U2 74141-SOCKET, U3 74HCT08

Commit message: Added info in silk
Other:
- note added: "Example: 2 pieces of Samtec TS-108-G-A"
Changed lines of the file:
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@@
+		)
+	)
+	(text "Example: 2 pieces of Samtec TS-108-G-A"
+		(exclude_from_sim no)
+		(at 124.714 46.99 0)
+		(effects
+			(font
+				(size 1.27 1.27)
+			)
 		)
 	)
@@
 		)
 		(property "Value" "74141-SOCKET"
-			(at 103.124 48.768 0)
-			(effects
-				(font
+			(at 103.124 43.942 0)
+			(effects
+				(font
